File: breadboard-offsetgain.kicad_sch (KiCad schematic)
At the start: 15 parts, among them J1 Conn_02x01, J2 Conn_02x01, J3 Conn_02x01, J4 Conn_02x01, J5 Conn_01x04, J6 Conn_01x04, U1 TL072

Commit message: Add image and schematic
Parts:
- removed J3, J4: Conn_02x01, Connector_PinHeader_2.54mm:PinHeader_2x01_P2.54mm_Vertical, symbol Connector_Generic:Conn_02x01
- J1, J2: value Conn_02x01 -> Conn_02x05; footprint Connector_PinHeader_2.54mm:PinHeader_2x01_P2.54mm_Vertical -> Connector_PinHeader_2.54mm:PinHeader_2x05_P2.54mm_Vertical; symbol Connector_Generic:Conn_02x01 -> Connector_Generic:Conn_02x05_Odd_Even
Connections:
- net +12V: now also J1.3 (Pin_3), J1.5 (Pin_5), J1.7 (Pin_7), J1.9 (Pin_9)
- net -12V: now also J2.3 (Pin_3), J2.5 (Pin_5), J2.7 (Pin_7), J2.9 (Pin_9)
- net GND: now also J1.10 (Pin_10), J1.4 (Pin_4), J1.6 (Pin_6), J1.8 (Pin_8), J2.10 (Pin_10), J2.4 (Pin_4), J2.6 (Pin_6), J2.8 (Pin_8)
Other:
- moved on the sheet: C1, C2, J5, J6, R1, R2, R3, R4, R5, R6, U1A, U1B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
